Commit message: add mid360

File: quadruped_descriptions/go2_description/xacro/robot.xacro (robot description, xacro)
@@ -7,4 +7,5 @@
   <xacro:include filename="$(find go2_description)/xacro/materials.xacro"/>
   <xacro:include filename="$(find go2_description)/xacro/leg.xacro"/>
+  <xacro:include filename="$(find go2_description)/model/mid360/mid360.xacro"/>
   <xacro:if value="$(arg GAZEBO)">
     <xacro:if value="$(arg CLASSIC)">
@@ -109,20 +110,7 @@
     </collision>
   </link>
-  <joint name="camera_joint_front" type="fixed">
-    <parent link="trunk"/>
-    <child link="front_camera"/>
-    <origin rpy="0 0 0" xyz="0.32715 0 0.04297"/>
-  </joint>
-  <link name="front_camera">
-  </link>
-  <joint name="lidar_joint" type="fixed">
-    <origin
-        xyz="0.28945 0 -0.046825" rpy="0 2.8782 0"/>
-    <parent link="trunk"/>
-    <child link="lidar"/>
-    <axis xyz="0 0 0"/>
-  </joint>
-  <link name="lidar">
-  </link>
+  <xacro:mid360  name="livox_frame" parent="trunk" topic="/livox">
+    <origin xyz="0.22 0.0 0.12" rpy="0.0 0 0.0"/>
+  </xacro:mid360>
   <xacro:leg name="FR" mirror="-1" mirror_dae="False" front_hind="1" front_hind_dae="True"/>
   <xacro:leg name="FL" mirror="1" mirror_dae="True" front_hind="1" front_hind_dae="True"/>

Commit message: reverse launch

File: quadruped_descriptions/go2_description/xacro/robot.xacro (robot description, xacro)
@@ -7,5 +7,4 @@
   <xacro:include filename="$(find go2_description)/xacro/materials.xacro"/>
   <xacro:include filename="$(find go2_description)/xacro/leg.xacro"/>
-  <xacro:include filename="$(find go2_description)/model/mid360/mid360.xacro"/>
   <xacro:if value="$(arg GAZEBO)">
     <xacro:if value="$(arg CLASSIC)">
@@ -50,12 +49,6 @@
         <mesh filename="file://$(find go2_description)/meshes/trunk.dae" scale="1 1 1"/>
       </geometry>
-      <!-- <material name="orange"/> -->
     </visual>
-    <collision>
-      <origin rpy="0 0 0" xyz="0 0 0"/>
-      <geometry>
-        <box size="${trunk_length} ${trunk_width} ${trunk_height}"/>
-      </geometry>
-    </collision>
+    <!-- 删除 mesh collision，避免巨大黑色实体 -->
     <collision>
       <origin rpy="0 0 0" xyz="0 0 0"/>
@@ -110,7 +103,16 @@
     </collision>
   </link>
-  <xacro:mid360  name="livox_frame" parent="trunk" topic="/livox">
-    <origin xyz="0.22 0.0 0.12" rpy="0.0 0 0.0"/>
-  </xacro:mid360>
+  <link name="livox_frame">
+    <visual>
+      <geometry>
+        <sphere radius="0.01"/> <!-- 用来占位 -->
+      </geometry>
+    </visual>
+  </link>
+  <joint name="livox_mount_joint" type="fixed">
+    <parent link="trunk"/>
+    <child link="livox_frame"/>
+    <origin xyz="0.22 0.0 0.12" rpy="0 0 0"/>
+  </joint>
   <xacro:leg name="FR" mirror="-1" mirror_dae="False" front_hind="1" front_hind_dae="True"/>
   <xacro:leg name="FL" mirror="1" mirror_dae="True" front_hind="1" front_hind_dae="True"/>
